File: 1. RAIDEN/PCB/PCB Sensores/PCB Sensores/PCB Sensores.kicad_pcb (KiCad board)
At the start: 2 copper layers, 72 x 105 mm, 32 parts, among them U1 BOB-09056

Commit message: Resistor Corrijido
Parts:
- moved R1 10.5 mm to (138.5, 69.2), turned to -90 degrees
Connections:
- R1 pad 2: SDA -> SCL
Routing:
- net SDA: track 28.1 -> 14.2 mm
- net VIN: track 314.2 -> 302.2 mm
- net SCL: track 255.8 -> 251.8 mm

Commit message: PCB Sesnores final
Parts:
- removed R10, R11, R12, R13, R3, R4, R5, R6, R7, R8, R9: R, Resistor_THT:R_Axial_DIN0207_L6.3mm_D2.5mm_P7.62mm_Horizontal
- moved R2 67.0 mm to (156.5, 95.3), turned to 90 degrees
Connections:
- R2 pad 2: SDA_1 -> SDA
Routing:
- net SCL: track 251.8 -> 229.9 mm
- net VIN: track 302.2 -> 290.6 mm
- net SDA_11: track 42.6 -> 37.2 mm
- net SDA_1: track 22.8 -> 17.3 mm
- net SDA_9: track 46.7 -> 41.3 mm
- net SDA_8: track 56.5 -> 51.1 mm
- net SDA_2: track 19.8 -> 14.3 mm
- net SDA_10: track 42.9 -> 37.5 mm
- net SDA: track 14.2 -> 18.9 mm
- net SDA_6: track 36.4 -> 34.6 mm
- net SDA_5: track 29.6 -> 27.8 mm
- net SDA_4: track 22.8 -> 21.0 mm
- net SDA_3: track 18.8 -> 17.0 mm
- net SDA_7: track 42.6 -> 40.8 mm
- net SDA_12: track 41.1 -> 39.3 mm
Other:
- board size 72 x 105 mm -> 75 x 105 mm
