File: 1. RAIDEN/PCB/PCB Sensores/PCB Sensores/PCB Sensores.kicad_sch (KiCad schematic)
At the start: 32 parts, among them U1 BOB-09056

Commit message: Resistor Corrijido
Connections:
- net SCL: now also R1.2
- net SDA: no longer R1.2
Other:
- moved on the sheet: R1
Changed lines of the file:
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@@
 	)
 	(junction
-		(at 191.77 59.69)
-		(diameter 0)
-		(color 0 0 0 0)
-	)
-	(junction
 		(at 152.4 109.22)
 		(diameter 0)
@@
 	(wire
 		(pts
-			(xy 191.77 60.96) (xy 191.77 59.69)
+			(xy 205.74 63.5) (xy 205.74 59.69)
 		)
 		(stroke
@@
 	(wire
 		(pts
-			(xy 191.77 68.58) (xy 191.77 71.12)
+			(xy 205.74 71.12) (xy 205.74 76.2)
 		)
 		(stroke
@@
 	(global_label "VIN"
 		(shape input)
-		(at 191.77 71.12 0)
+		(at 205.74 76.2 0)
 		(fields_autoplaced yes)
 		(effects
@@
 		)
 		(property "Intersheetrefs" "${INTERSHEET_REFS}"
-			(at 197.8742 71.12 0)
+			(at 211.8442 76.2 0)
 			(hide yes)
 			(show_name no)
@@
 	(global_label "SDA"
 		(shape input)
-		(at 198.12 57.15 270)
+		(at 195.58 57.15 270)
 		(fields_autoplaced yes)
 		(effects
@@
 		)
 		(property "Intersheetrefs" "${INTERSHEET_REFS}"
-			(at 198.12 63.7033 90)
+			(at 195.58 63.7033 90)
 			(hide yes)
 			(show_name no)
@@
 	(symbol
 		(lib_id "Device:R")
-		(at 191.77 64.77 180)
+		(at 205.74 67.31 180)
 		(unit 1)
 		(body_style 1)
@@
 		(fields_autoplaced yes)
 		(property "Reference" "R1"
-			(at 194.31 63.4999 0)
+			(at 208.28 66.0399 0)
 			(show_name no)
 			(do_not_autoplace no)
@@
 		)
 		(property "Value" "R"
-			(at 194.31 66.0399 0)
+			(at 208.28 68.5799 0)
 			(show_name no)
 			(do_not_autoplace no)
@@
 		)
 		(property "Footprint" "Resistor_THT:R_Axial_DIN0207_L6.3mm_D2.5mm_P7.62mm_Horizontal"
-			(at 193.548 64.77 90)
+			(at 207.518 67.31 90)
 			(hide yes)
 			(show_name no)
@@
 		)
 		(property "Datasheet" ""
-			(at 191.77 64.77 0)
+			(at 205.74 67.31 0)
 			(hide yes)
 			(show_name no)
@@
 		)
 		(property "Description" "Resistor"
-			(at 191.77 64.77 0)
+			(at 205.74 67.31 0)
 			(hide yes)
 			(show_name no)

Commit message: PCB Sesnores final
Parts:
- removed R10, R11, R12, R13, R3, R4, R5, R6, R7, R8, R9: R, Resistor_THT:R_Axial_DIN0207_L6.3mm_D2.5mm_P7.62mm_Horizontal, symbol Device:R
Connections:
- net SDA: now also R2.2
- net SDA_1: no longer R2.2
